File: peripherals.sch (KiCad schematic (older format))
At the start: 4 parts

Commit message: 20191113未完工
Parts:
- removed D?: LED_ARGB, symbol Device:LED_ARGB
- added C21, C23, C25: 0603_10uF__106_10%_10V, lc_lib:0603_C, symbol lc_Cap:0603_10uF__106_10%_10V
- added C22, C24, C26: 0603_100nF__104_10%_50V, lc_lib:0603_C, symbol lc_Cap:0603_100nF__104_10%_50V
- added J13: Conn_01x03_Male, symbol Connector:Conn_01x03_Male
- added J14: Conn_01x14_Female, symbol Connector:Conn_01x14_Female
- added R21, R22, R23, R24, R25, R26, R27, R34, R40, R41, R42, R43, R44, R45, R46, R47, R48, R49, R50, R51, R52: 0603_0Ω__0R0_1%, lc_lib:0603_R, symbol lc_RES:0603_0Ω__0R0_1%
- added R29, R30, R31, R32, R33, R38, R39: 0603_10KΩ__1002_1%, lc_lib:0603_R, symbol lc_RES:0603_10KΩ__1002_1%
- added U6: MPU-6050, Sensor_Motion:InvenSense_QFN-24_4x4mm_P0.5mm, symbol Sensor_Motion:MPU-6050
- added U?: TM1638_[C19187], lc_lib:SOIC-28_300MIL, symbol lc_IC:TM1638_[C19187]
- gave numbers to parts that had none: 3
Connections:
- net labels added: +3V3, LCD_BL, LCD_CS, LCD_DAT\CON, LCD_D\C, LCD_MISO, LCD_MOSI, LCD_RST, LCD_SCK, LCD_VCC, SD_DET, TCH_CS, TCH_IRQ, TCH_MISO, TCH_MOSI, TCH_SCK
- wire segments 21 -> 86
- no-connect marks 1 -> 2
Other:
- note added: "Female"
- note added: "Not yet determined."
- note removed: "C404284"
- moved on the sheet: J11, R28

Commit message: 20191113
Parts:
- removed C21, C23, C25: 0603_10uF__106_10%_10V, lc_lib:0603_C, symbol lc_Cap:0603_10uF__106_10%_10V
- removed C22, C24, C26: 0603_100nF__104_10%_50V, lc_lib:0603_C, symbol lc_Cap:0603_100nF__104_10%_50V
- removed J11: Conn_02x09_Odd_Even, symbol Connector_Generic:Conn_02x09_Odd_Even
- removed J12: Micro_SD_Card_Det, symbol Connector:Micro_SD_Card_Det
- removed J13: Conn_01x03_Male, symbol Connector:Conn_01x03_Male
- removed J14: Conn_01x14_Female, symbol Connector:Conn_01x14_Female
- removed R21, R22, R23, R24, R25, R26, R27, R34, R40, R41, R42, R43, R44, R45, R46, R47, R48, R49, R50, R51, R52: 0603_0Ω__0R0_1%, lc_lib:0603_R, symbol lc_RES:0603_0Ω__0R0_1%
- removed R28, R29, R30, R31, R32, R33, R38, R39: 0603_10KΩ__1002_1%, lc_lib:0603_R, symbol lc_RES:0603_10KΩ__1002_1%
Connections:
- net labels removed: +3.3V, +3V3, GND, LCD_BL, LCD_CS, LCD_DAT\CON, LCD_D\C, LCD_MISO, LCD_MOSI, LCD_RST, LCD_SCK, LCD_VCC, OV_D0, OV_D1, OV_D2, OV_D3, OV_D4, OV_D5, OV_D6, OV_D7, OV_HREF, OV_PCLK, OV_PWDN, OV_RESET, OV_SCL, OV_SDA, OV_VSYNC, SD_CLK, SD_CMD, SD_D0, SD_D1, SD_D2, SD_D3, SD_DET, TCH_CS, TCH_IRQ, TCH_MISO, TCH_MOSI, TCH_SCK
- wire segments 86 -> 0
- no-connect marks 2 -> 0
Other:
- note removed: "Female"
- note removed: "Not yet determined."
