File: MyESP32EvalBoard.kicad_pcb (KiCad board)
At the start: 2 copper layers, 94 parts, among them J1 Conn_01x19_Male, J11 Conn_02x09_Odd_Even, J12 Conn_01x14_Female, J2 Conn_01x19_Male, J3 Conn_01x02_Male, J4 Conn_01x02_Male, J5 Conn_01x02_Male, J6 Conn_01x02_Male, J7 Conn_ARM_JTAG_SWD_20, J8 HR911105A, J9 USB_C_Receptacle_USB2.0, U1 ESP32-WROVER, U2 ESP32-WROOM-32D, U3 PCA9535PW, U4 LAN8720A, U5 AOZ1031, U6 SRV05-4-P-T7_[C85364], U7 CH340G, U8 MPU-6050, U9 BMP280, Y1 SMD-3225_4P__25MHZ_12PF_10PPM, Y2 SMD-3225_4P__12MHZ_20PF_10PPM

Commit message: 20191114
Parts:
- removed the C15 at (-132.5, 50.5)
- removed the C16 at (-127.5, 65.2)
- removed C18: 0603_100nF__104_10%_50V, lc_lib:0603_C
- removed J12: Conn_01x14_Female, Connector_PinSocket_2.54mm:PinSocket_1x14_P2.54mm_Vertical
- removed J4, J5, J6: Conn_01x02_Male, Connector_PinHeader_2.54mm:PinHeader_1x02_P2.54mm_Vertical
- removed the J7 at (-118.1, 0.00)
- removed the R19 at (-129.5, 47.7)
- removed the R21 at (144.9, 0.89)
- removed the R22 at (149.2, 3.67)
- removed the R23 at (144.9, 3.67)
- removed the R25 at (144.9, 6.45)
- removed the R27 at (-39.3, 57.7)
- removed the R28 at (-35.0, 57.7)
- removed R29, R30, R31, R32, R33, R34, R35, R36, R37, R38, R39: 0603_0Ω__0R0_1%, lc_lib:0603_R
- removed the R8 at (34.6, 17.9)
- removed the U4 at (35.6, -0.21)
- removed the U6 at (-129.1, 56.6)
- added C13: 0603_1uF__105_10%_50V, lc_lib:0603_C, F.Cu at (165.8, 42.5)
- added C23: 0603_100nF__104_10%_50V, lc_lib:0603_C, F.Cu at (105.5, 9.00)
- added C24: 0603_100nF__104_10%_50V, lc_lib:0603_C, F.Cu at (72.5, 45.4)
- added C25: 0603_100nF__104_10%_50V, lc_lib:0603_C, F.Cu at (64.0, 42.6)
- added C29: 0603_100nF__104_10%_50V, lc_lib:0603_C, F.Cu at (12.2, 65.2)
- added C30: 3.3uF, Capacitor_SMD:CP_Elec_4x5.4, F.Cu at (36.2, 47.0)
- added C33: 0603_100nF__104_10%_50V, lc_lib:0603_C, F.Cu at (30.8, 56.2)
- added C34: 0603_1uF__105_10%_50V, lc_lib:0603_C, F.Cu at (30.8, 58.0)
- added C35: 3.3uF, Capacitor_SMD:CP_Elec_4x5.4, F.Cu at (24.2, 56.2)
- added C36: 3.3uF, Capacitor_SMD:CP_Elec_4x5.4, F.Cu at (24.2, 51.2)
- added C37: 0603_1uF__105_10%_50V, lc_lib:0603_C, F.Cu at (16.2, 50.5)
- added C38: 0603_1uF__105_10%_50V, lc_lib:0603_C, F.Cu at (16.2, 57.0)
- added C6: 0805_22uF__226_20%_25V, lc_lib:0805_C, F.Cu at (152.5, 33.5)
- added C7: 0805_22uF__226_20%_25V, lc_lib:0805_C, F.Cu at (150.2, 33.5)
- added C8: 0603_1uF__105_10%_50V, lc_lib:0603_C, F.Cu at (154.5, 33.6)
- added C9: 0603_100nF__104_10%_50V, lc_lib:0603_C, F.Cu at (156.3, 33.6)
- added H1: MountingHole_Pad, MountingHole:MountingHole_3.2mm_M3_Pad, F.Cu at (15.0, 6.00)
- added H2: MountingHole_Pad, MountingHole:MountingHole_3.2mm_M3_Pad, F.Cu at (24.0, 66.0)
- added H3: MountingHole_Pad, MountingHole:MountingHole_3.2mm_M3_Pad, F.Cu at (138.0, 66.0)
- added H4: MountingHole_Pad, MountingHole:MountingHole_3.2mm_M3_Pad, F.Cu at (138.0, 12.0)
- added J10: Conn_01x14_Female, Connector_PinSocket_2.54mm:PinSocket_1x14_P2.54mm_Vertical, F.Cu at (104.0, 4.00)
- added L1: 4.7uH, Inductor_SMD:L_7.3x7.3_H3.5, F.Cu at (158.6, 48.1)
- added LS1: Speaker, Connector_PinHeader_2.54mm:PinHeader_1x02_P2.54mm_Vertical, F.Cu at (13.0, 56.2)
- added LS2: Speaker, Connector_PinHeader_2.54mm:PinHeader_1x02_P2.54mm_Vertical, F.Cu at (13.0, 51.2)
- added R13: 0603_0Ω__0R0_1%, lc_lib:0603_R, F.Cu at (125.1, 8.50)
- added R14: 0603_0Ω__0R0_1%, lc_lib:0603_R, F.Cu at (102.2, 9.00)
- added R15: 0603_10KΩ__1002_1%, lc_lib:0603_R, F.Cu at (19.5, 59.0)
- added R16: 0603_10KΩ__1002_1%, lc_lib:0603_R, F.Cu at (19.5, 48.5)
- added R17: 0603_470Ω__4700_1%, lc_lib:0603_R, F.Cu at (18.8, 56.2)
- added R18: 0603_470Ω__4700_1%, lc_lib:0603_R, F.Cu at (18.8, 51.2)
- added R9: 0603_1KΩ__1001_1%, lc_lib:0603_R, F.Cu at (175.5, 34.8)
- added U10: LAN8720A, Package_DFN_QFN:QFN-24-1EP_4x4mm_P0.5mm_EP2.6x2.6mm, F.Cu at (28.0, 35.0)
- added U5: SRV05-4, Package_TO_SOT_SMD:SOT-23-6, F.Cu at (130.0, 22.2)
- added U9: CS4344, Package_SO:TSSOP-10_3x3mm_P0.5mm, F.Cu at (32.2, 53.5)
- C17: value 0603_1uF__105_10%_50V -> 0603_20pF__200_5%_50V
- C22: value 0603_1uF__105_10%_50V -> 0603_10uF__106_10%_10V
- C26: value 0603_20pF__200_5%_50V -> 0603_100nF__104_10%_50V
- C27: value 0603_10uF__106_10%_10V -> 0603_2.2nF__222_10%_50V
- C31: value 0603_10uF__106_10%_10V -> 0603_100nF__104_10%_50V
- C32: value 0603_100nF__104_10%_50V -> 10uF; footprint lc_lib:0603_C -> Capacitor_SMD:CP_Elec_4x5.3
- J3: value Conn_01x02_Male -> Conn_01x06_Male; footprint Connector_PinHeader_2.54mm:PinHeader_1x02_P2.54mm_Vertical -> Connector_PinHeader_2.54mm:PinHeader_1x06_P2.54mm_Vertical
- R24: value 0603_0Ω__0R0_1% -> 0603_49.9Ω__49R9_1%
- moved R8 310.8 mm to (166.5, 45.0), turned to 0 degrees
- moved D1 308.6 mm to (175.5, 38.8), turned to 270 degrees
- moved C11 305.9 mm to (162.0, 42.3)
- moved R10 305.6 mm to (167.5, 42.5)
- moved C12 299.4 mm to (164.0, 42.5)
- moved U4 287.8 mm to (154.5, 40.2), turned to 270 degrees
- moved R6 286.4 mm to (150.2, 37.4), turned to 0 degrees
- moved J7 283.5 mm to (139.2, 22.0)
- moved R7 283.0 mm to (150.2, 39.3), turned to 180 degrees
- moved C10 282.7 mm to (150.2, 41.2), turned to 0 degrees
- moved R5 279.8 mm to (150.2, 43.1), turned to 180 degrees
- moved R3 274.9 mm to (133.8, 24.5), turned to 180 degrees
- moved R4 273.9 mm to (133.9, 20.2), turned to 180 degrees
- moved Y1 273.5 mm to (128.8, 16.2)
- moved C14 273.4 mm to (131.5, 16.5)
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- renumbered C19 to C10, C20 to C11, C21 to C12, C23 to C14, C24 to C15, C25 to C16, C29 to C20, C30 to C21, C6 to C39, C7 to C40, C8 to C41, C9 to C42, C10 to C43, C11 to C44, C12 to C45, C13 to C46, C14 to C47, J8 to J11, J9 to J7, J11 to J9, R20 to R10, R26 to R12, R3 to R19, R4 to R20, R5 to R21, R6 to R22, R7 to R23, R9 to R25, R10 to R26, R11 to R27, R12 to R28, R13 to R3, R14 to R4, R15 to R5, R16 to R6, R17 to R7, R18 to R8, U5 to U4, U7 to U6, U8 to U7, U9 to U8, Y2 to Y1, Y1 to Y2
Connections:
- C11 pad 1: Net-(C20-Pad1) -> Net-(C11-Pad1)
- C12 pad 1: Net-(C20-Pad1) -> Net-(C11-Pad1)
- C17 pad 1: VBUS -> Net-(C17-Pad1)
- C22 pad 1: Net-(C20-Pad1) -> GND
- C22 pad 2: GND -> /SPI LCD and Touch/LCD_VCC
- C28 pad 1: Net-(C27-Pad1) -> VDD
- C31 pad 1: GND -> Net-(C30-Pad1)
- C31 pad 2: VDD -> GND
- C32 pad 1: GND -> Net-(C32-Pad1)
- C32 pad 2: VDD -> GND
- J1 pad 2: /ESP32MCU/ESP32_VDD -> VDD
- J2 pad 11: /ESP32MCU/ESP32_IO16 -> /ESP32MCU/ESP32_IO17
- J2 pad 12: /ESP32MCU/ESP32_IO17 -> /ESP32MCU/ESP32_IO16
- J2 pad 4: /ESP32MCU/UART_TXD -> /Power and USB UART/RXD
- J2 pad 5: /ESP32MCU/UART_RXD -> /Power and USB UART/TXD
- J3 pad 1: Net-(J3-Pad1) -> VDD
- J3 pad 2: /ESP32MCU/ESP32_IO12 -> /ESP32MCU/ESP32_IO14
- J7 pad A4: Net-(J9-PadA4) -> VBUS
- J7 pad A8: Net-(J9-PadA8) -> (no net)
- J7 pad A9: Net-(J9-PadA4) -> VBUS
- J7 pad B4: Net-(J9-PadA4) -> VBUS
- J7 pad B8: Net-(J9-PadB8) -> (no net)
- J7 pad B9: Net-(J9-PadA4) -> VBUS
- J9 pad 10: /CAMERA OV2640/OV_D1 -> (no net)
- J9 pad 11: /CAMERA OV2640/OV_D4 -> (no net)
- J9 pad 12: /CAMERA OV2640/OV_D3 -> (no net)
- J9 pad 13: /CAMERA OV2640/OV_D6 -> (no net)
- J9 pad 14: /CAMERA OV2640/OV_D5 -> (no net)
- J9 pad 15: /CAMERA OV2640/OV_PCLK -> (no net)
- J9 pad 16: /CAMERA OV2640/OV_D7 -> (no net)
- J9 pad 18: Net-(J11-Pad18) -> (no net)
- J9 pad 3: /CAMERA OV2640/OV_SCL -> I2C_SCL
- J9 pad 4: /CAMERA OV2640/OV_VSYNC -> (no net)
- J9 pad 5: /CAMERA OV2640/OV_SDA -> I2C_SDA
- J9 pad 6: /CAMERA OV2640/OV_HREF -> (no net)
- J9 pad 7: /CAMERA OV2640/OV_D0 -> (no net)
- J9 pad 8: /CAMERA OV2640/OV_RESET -> (no net)
- J9 pad 9: /CAMERA OV2640/OV_D2 -> (no net)
- R24 pad 1: /SD Card/SD_SCK -> VDDA
- R24 pad 2: Net-(J10-Pad5) -> /Ethernet/ETH_TX-
- R26 pad 1: +3V3 -> VDDA
- R6 pad 1: Net-(C20-Pad1) -> Net-(C11-Pad1)
- R8 pad 1: Net-(C20-Pad1) -> Net-(C11-Pad1)
- U1 pad 27: /ESP32MCU/ESP32_IO17 -> /ESP32MCU/ESP32_IO16
- U1 pad 28: /ESP32MCU/ESP32_IO16 -> /ESP32MCU/ESP32_IO17
- U1 pad 32: Net-(U1-Pad32) -> (no net)
- U1 pad 34: /ESP32MCU/UART_RXD -> /Power and USB UART/TXD
- U1 pad 35: /ESP32MCU/UART_TXD -> /Power and USB UART/RXD
- U2 pad 32: Net-(U2-Pad32) -> (no net)
- U2 pad 34: /ESP32MCU/UART_RXD -> /Power and USB UART/TXD
- U2 pad 35: /ESP32MCU/UART_TXD -> /Power and USB UART/RXD
- U3 pad 1: /ESP32MCU/ESP32_GPIO36 -> (no net)
- U3 pad 10: /ESP32MCU/EXT_IO6 -> (no net)
- U3 pad 11: /ESP32MCU/EXT_IO7 -> (no net)
- U3 pad 13: /ESP32MCU/EXT_IO10 -> (no net)
- U3 pad 14: /ESP32MCU/EXT_IO11 -> (no net)
- U3 pad 15: /ESP32MCU/EXT_IO12 -> (no net)
- U3 pad 16: /ESP32MCU/EXT_IO13 -> (no net)
- U3 pad 17: /ESP32MCU/EXT_IO14 -> (no net)
- U3 pad 18: /ESP32MCU/EXT_IO15 -> (no net)
- U3 pad 19: /ESP32MCU/EXT_IO16 -> (no net)
- U3 pad 2: Net-(U3-Pad2) -> (no net)
- U3 pad 20: /ESP32MCU/EXT_IO17 -> (no net)
- U3 pad 21: Net-(U3-Pad21) -> (no net)
- U3 pad 22: /ESP32MCU/I2C_SCL -> I2C_SCL
- U3 pad 23: /ESP32MCU/I2C_SDA -> I2C_SDA
- U3 pad 3: Net-(U3-Pad3) -> (no net)
- U3 pad 4: /ESP32MCU/EXT_IO0 -> (no net)
- U3 pad 5: /ESP32MCU/EXT_IO1 -> (no net)
- U3 pad 6: /ESP32MCU/EXT_IO2 -> (no net)
- U3 pad 7: /ESP32MCU/EXT_IO3 -> (no net)
- U3 pad 8: /ESP32MCU/EXT_IO4 -> (no net)
- U3 pad 9: /ESP32MCU/EXT_IO5 -> (no net)
- U6 pad 1: Net-(U7-Pad1) -> (no net)
- U6 pad 10: Net-(U7-Pad10) -> (no net)
- U6 pad 11: Net-(U7-Pad11) -> (no net)
- U6 pad 12: Net-(U7-Pad12) -> (no net)
- U6 pad 13: Net-(U7-Pad13) -> (no net)
- U6 pad 14: Net-(U7-Pad14) -> (no net)
- U6 pad 15: Net-(U7-Pad15) -> (no net)
- U6 pad 8: Net-(C26-Pad1) -> Net-(C17-Pad1)
- U6 pad 9: Net-(U7-Pad9) -> (no net)
- U7 pad 1: Net-(U8-Pad1) -> (no net)
- U7 pad 10: Net-(U8-Pad10) -> Net-(C26-Pad1)
- U7 pad 11: Net-(U8-Pad11) -> (no net)
- U7 pad 12: Net-(U8-Pad12) -> (no net)
- U7 pad 13: Net-(U8-Pad13) -> VDDA
- U7 pad 18: Net-(U8-Pad18) -> GND
- U7 pad 20: Net-(U8-Pad20) -> Net-(C27-Pad1)
- U7 pad 23: Net-(U8-Pad23) -> I2C_SCL
- U7 pad 24: Net-(U8-Pad24) -> I2C_SDA
- U7 pad 6: Net-(U8-Pad6) -> (no net)
- U7 pad 7: Net-(U8-Pad7) -> (no net)
- U7 pad 8: Net-(U8-Pad8) -> VDD
- U7 pad 9: Net-(U8-Pad9) -> GND
- U8 pad 1: Net-(U9-Pad1) -> GND
- U8 pad 2: Net-(U9-Pad2) -> VDD
- U8 pad 3: Net-(U9-Pad3) -> I2C_SDA
- U8 pad 4: Net-(U9-Pad4) -> I2C_SCL
- U8 pad 5: Net-(U9-Pad5) -> GND
- U8 pad 6: Net-(U9-Pad6) -> VDD
- U8 pad 7: Net-(U9-Pad7) -> GND
- U8 pad 8: Net-(U9-Pad8) -> VDDA
- Y1 pad 3: Net-(C26-Pad1) -> Net-(C17-Pad1)
Routing:
- net Net-(C40-Pad2): track 0.00 -> 13.9 mm
- net Net-(C41-Pad2): track 0.00 -> 10.9 mm
Other:
- board outline added: 135 x 72 mm
- copper layers 2 -> 4
