File: camera.sch (KiCad schematic (older format))
At the start: 4 parts, among them J11 Conn_02x09_Odd_Even

Commit message: 20191114
Parts:
- renumbered C29 to C20, C30 to C21, J11 to J9, R26 to R12
Changed lines of the file:
@@
 $Descr A4 11693 8268
 encoding utf-8
-Sheet 7 9
+Sheet 4 8
 Title ""
 Date ""
@@
 P 5800 3850
 AR Path="/5DF49590/5DCFB62F" Ref="J?"  Part="1"
-AR Path="/5DCEE55C/5DCFB62F" Ref="J11"  Part="1"
-F 0 "J11" H 5850 4467 50  0000 C CNN
+AR Path="/5DCEE55C/5DCFB62F" Ref="J9"  Part="1"
+F 0 "J9" H 5850 4467 50  0000 C CNN
 F 1 "Conn_02x09_Odd_Even" H 5850 4376 50  0000 C CNN
 F 2 "Connector_PinSocket_2.54mm:PinSocket_2x09_P2.54mm_Vertical" H 5800 3850 50  0001 C CNN
@@
 P 5600 3450
 AR Path="/5DF49590/5DCFB635" Ref="#PWR?"  Part="1"
-AR Path="/5DCEE55C/5DCFB635" Ref="#PWR060"  Part="1"
-F 0 "#PWR060" H 5600 3200 50  0001 C CNN
+AR Path="/5DCEE55C/5DCFB635" Ref="#PWR040"  Part="1"
+F 0 "#PWR040" H 5600 3200 50  0001 C CNN
 F 1 "GND" V 5605 3322 50  0000 R CNN
 F 2 "" H 5600 3450 50  0001 C CNN
@@
 P 4550 4450
 AR Path="/5DF49590/5DCFB658" Ref="R?"  Part="1"
-AR Path="/5DCEE55C/5DCFB658" Ref="R26"  Part="1"
-F 0 "R26" H 4550 4657 50  0000 C CNN
+AR Path="/5DCEE55C/5DCFB658" Ref="R12"  Part="1"
+F 0 "R12" H 4550 4657 50  0000 C CNN
 F 1 "0603_10KΩ__1002_1%" H 4400 4640 50  0001 L BNN
 F 2 "lc_lib:0603_R" H 4350 4210 50  0001 L BNN
@@
 P 4550 4650
 AR Path="/5DF49590/5DCFB65E" Ref="#PWR?"  Part="1"
-AR Path="/5DCEE55C/5DCFB65E" Ref="#PWR059"  Part="1"
-F 0 "#PWR059" H 4550 4400 50  0001 C CNN
+AR Path="/5DCEE55C/5DCFB65E" Ref="#PWR039"  Part="1"
+F 0 "#PWR039" H 4550 4400 50  0001 C CNN
 F 1 "GND" H 4555 4477 50  0000 C CNN
 F 2 "" H 4550 4650 50  0001 C CNN
@@
 P 6700 2950
 AR Path="/5DF49590/5DCFB68A" Ref="C?"  Part="1"
-AR Path="/5DCEE55C/5DCFB68A" Ref="C29"  Part="1"
-F 0 "C29" V 7004 3060 50  0000 L CNN
+AR Path="/5DCEE55C/5DCFB68A" Ref="C20"  Part="1"
+F 0 "C20" V 7004 3060 50  0000 L CNN
 F 1 "0603_10uF__106_10%_10V" H 6749 3180 50  0001 L BNN
 F 2 "lc_lib:0603_C" H 6699 2670 50  0001 L BNN
@@
 P 6900 2950
 AR Path="/5DF49590/5DCFB697" Ref="C?"  Part="1"
-AR Path="/5DCEE55C/5DCFB697" Ref="C30"  Part="1"
-F 0 "C30" V 7204 3060 50  0000 L CNN
+AR Path="/5DCEE55C/5DCFB697" Ref="C21"  Part="1"
+F 0 "C21" V 7204 3060 50  0000 L CNN
 F 1 "0603_100nF__104_10%_50V" H 6949 3180 50  0001 L BNN
 F 2 "lc_lib:0603_C" H 6899 2670 50  0001 L BNN
@@
 P 6900 3150
 AR Path="/5DF49590/5DCFB6A2" Ref="#PWR?"  Part="1"
-AR Path="/5DCEE55C/5DCFB6A2" Ref="#PWR062"  Part="1"
-F 0 "#PWR062" H 6900 2900 50  0001 C CNN
+AR Path="/5DCEE55C/5DCFB6A2" Ref="#PWR042"  Part="1"
+F 0 "#PWR042" H 6900 2900 50  0001 C CNN
 F 1 "GND" V 6905 3022 50  0000 R CNN
 F 2 "" H 6900 3150 50  0001 C CNN
@@
 	6350 3450 6700 3450
 $Comp
-L power:VDD #PWR061
+L power:VDD #PWR041
 U 1 1 5DD2C3AD
 P 6350 3000
-F 0 "#PWR061" H 6350 2850 50  0001 C CNN
+F 0 "#PWR041" H 6350 2850 50  0001 C CNN
 F 1 "VDD" H 6367 3173 50  0000 C CNN
 F 2 "" H 6350 3000 50  0001 C CNN
