File: esp32mcu.sch (KiCad schematic (older format))
At the start: 3 parts

Commit message: 20191112未完成的工作
Parts:
- removed J?: Conn_02x09_Odd_Even, symbol Connector_Generic:Conn_02x09_Odd_Even
- removed R?: 0603_10KΩ__1002_1%, lc_lib:0603_R, symbol lc_RES:0603_10KΩ__1002_1%
- added C?: 0603_100nF__104_10%_50V, lc_lib:0603_C, symbol lc_Cap:0603_100nF__104_10%_50V
- added C? (x2): 0603_1uF__105_10%_50V, lc_lib:0603_C, symbol lc_Cap:0603_1uF__105_10%_50V
- added R?: 0603_0Ω__0R0_1%, lc_lib:0603_R, symbol lc_RES:0603_0Ω__0R0_1%
- added R?: 0603_10KΩ__1002_1%, lc_lib:0603_R, symbol lc_RES:0603_10KΩ__1002_1%
- added Touch? (x4): TouchPoint, symbol Connector:TestPoint
- added U?: ESP32-WROOM-32D, RF_Module:ESP32-WROOM-32, symbol RF_Module:ESP32-WROOM-32D
Connections:
- net labels added: +3V3, ESP32_3V3, ESP32_EN, ESP32_IO0, ESP32_IO10, ESP32_IO11, ESP32_IO12, ESP32_IO13, ESP32_IO14, ESP32_IO15, ESP32_IO16, ESP32_IO17, ESP32_IO18, ESP32_IO19, ESP32_IO2, ESP32_IO21, ESP32_IO22, ESP32_IO23, ESP32_IO25, ESP32_IO26, ESP32_IO27, ESP32_IO32, ESP32_IO33, ESP32_IO34, ESP32_IO35, ESP32_IO36, ESP32_IO39, ESP32_IO4, ESP32_IO5, ESP32_IO6, ESP32_IO7, ESP32_IO8, ESP32_IO9, ESP32_RXD, ESP32_TXD, UART_RXD, UART_TXD
- net labels removed: +3.3V, OV_D0, OV_D1, OV_D2, OV_D3, OV_D4, OV_D5, OV_D6, OV_D7, OV_HREF, OV_PCLK, OV_PWDN, OV_RESET, OV_SCL, OV_SDA, OV_VSYNC
- wire segments 15 -> 84
- no-connect marks 1 -> 0
Other:
- note added: "GPIO16&17 not exist in ESP32-WROVER."
- moved on the sheet: U?

Commit message: 20191113未完工
Parts:
- removed Touch? (x4): TouchPoint, symbol Connector:TestPoint
- added J8, J9: Conn_01x19_Male, symbol Connector:Conn_01x19_Male
- gave numbers to parts that had none: 7
Connections:
- net labels added: ESP32_VDD, VDD
- net labels removed: +3V3, ESP32_3V3
- wire segments 84 -> 114

Commit message: 20191113
Parts:
- added C4: 0603_1uF__105_10%_50V, lc_lib:0603_C, symbol lc_Cap:0603_1uF__105_10%_50V
- added C5: 0603_100nF__104_10%_50V, lc_lib:0603_C, symbol lc_Cap:0603_100nF__104_10%_50V
- added J3, J4, J5, J6: Conn_01x02_Male, Connector_PinHeader_2.54mm:PinHeader_1x02_P2.54mm_Vertical, symbol Connector:Conn_01x02_Male
- added J7: Conn_ARM_JTAG_SWD_20, Connector_PinSocket_2.54mm:PinSocket_2x10_P2.54mm_Vertical, symbol Connector:Conn_ARM_JTAG_SWD_20
- added U3: PCA9535PW, Package_SO:TSSOP-24_4.4x7.8mm_P0.65mm, symbol Interface_Expansion:TCA9535PWR
- J1: renamed from J8; footprint (none) -> Connector_PinHeader_2.54mm:PinHeader_1x19_P2.54mm_Vertical
- J2: renamed from J9; footprint (none) -> Connector_PinHeader_2.54mm:PinHeader_1x19_P2.54mm_Vertical
- U1: renamed from U3; footprint (none) -> esp32-wrover:ESP32-WROVER
- renumbered C9 to C1, C10 to C2, C11 to C3, R9 to R1, R10 to R2, U4 to U2
Connections:
- net ESP32_IO12: now also J3.2 (Pin_2)
- net ESP32_IO13: now also J6.2 (Pin_2)
- net ESP32_IO14: now also J5.2 (Pin_2)
- net ESP32_IO15: now also J4.2 (Pin_2)
- net GND: now also C4.1, C5.1, J7.10 (GND), J7.12 (GND), J7.14 (GND), J7.16 (GND), J7.18 (GND), J7.20 (GND), J7.4 (GND), J7.6 (GND), J7.8 (GND), U3.12 (GND)
- net VDD: now also C4.2, C5.2, J7.1 (VTREF), U3.24 (VCC)
- new net: J3.1 (Pin_1), J7.5 (TDI)
- new net: J6.1 (Pin_1), J7.9 (TCK/SWDCLK)
- new net: J5.1 (Pin_1), J7.7 (TMS/SWDIO)
- new net: J4.1 (Pin_1), J7.13 (TDO/SWO)
- new net ESP32_GPIO36: U3.1 (~INT)
- new net EXT_IO0: U3.4 (P00)
- new net EXT_IO1: U3.5 (P01)
- new net EXT_IO10: U3.13 (P10)
- new net EXT_IO11: U3.14 (P11)
- new net EXT_IO12: U3.15 (P12)
- new net EXT_IO13: U3.16 (P13)
- new net EXT_IO14: U3.17 (P14)
- new net EXT_IO15: U3.18 (P15)
- new net EXT_IO16: U3.19 (P16)
- new net EXT_IO17: U3.20 (P17)
- new net EXT_IO2: U3.6 (P02)
- new net EXT_IO3: U3.7 (P03)
- new net EXT_IO4: U3.8 (P04)
- new net EXT_IO5: U3.9 (P05)
- new net EXT_IO6: U3.10 (P06)
- new net EXT_IO7: U3.11 (P07)
- new net I2C_SCL: U3.22 (SCL)
- new net I2C_SDA: U3.23 (SDA)
- no-connect marks 0 -> 6
Other:
- moved on the sheet: J1, J2

Commit message: 20191114
Parts:
- removed J3, J4, J5, J6: Conn_01x02_Male, Connector_PinHeader_2.54mm:PinHeader_1x02_P2.54mm_Vertical, symbol Connector:Conn_01x02_Male
- removed J7: Conn_ARM_JTAG_SWD_20, Connector_PinSocket_2.54mm:PinSocket_2x10_P2.54mm_Vertical, symbol Connector:Conn_ARM_JTAG_SWD_20
- added J3: Conn_01x06_Male, Connector_PinHeader_2.54mm:PinHeader_1x06_P2.54mm_Vertical, symbol Connector:Conn_01x06_Male
Connections:
- net ESP32_IO12: now also J3.3 (Pin_3)
- net ESP32_IO13: now also J3.4 (Pin_4)
- net ESP32_IO14: now also J3.2 (Pin_2)
- net ESP32_IO15: now also J3.5 (Pin_5)
- net ESP32_IO16: now also J2.12 (Pin_12), U1.27 (IO16); no longer J2.11 (Pin_11), U1.28 (IO17)
- net ESP32_IO17: now also J2.11 (Pin_11), U1.28 (IO17); no longer J2.12 (Pin_12), U1.27 (IO16)
- net ESP32_VDD: no longer J1.2 (Pin_2)
- net GND: now also J3.6 (Pin_6)
- net VDD: now also J1.2 (Pin_2), J3.1 (Pin_1)
- no-connect marks 6 -> 0
Other:
- note added: "JTAG only for test in ver 0."
- note added: "MTCK"
- note added: "MTDI"
- note added: "MTDO"
- note added: "MTMS"
Changed lines of the file:
@@
 $Descr A4 11693 8268
 encoding utf-8
-Sheet 2 9
+Sheet 2 8
 Title ""
 Date ""
@@
 	3350 1350 3350 1250
 $Comp
-L power:GND #PWR011
+L power:GND #PWR012
 U 1 1 5DE9591C
 P 3350 1250
-F 0 "#PWR011" H 3350 1000 50  0001 C CNN
+F 0 "#PWR012" H 3350 1000 50  0001 C CNN
 F 1 "GND" V 3355 1122 50  0000 R CNN
 F 2 "" H 3350 1250 50  0001 C CNN
@@
 	5750 700  5050 700
 $Comp
-L power:GND #PWR012
+L power:GND #PWR013
 U 1 1 5DEC8C1F
 P 5750 3850
-F 0 "#PWR012" H 5750 3600 50  0001 C CNN
+F 0 "#PWR013" H 5750 3600 50  0001 C CNN
 F 1 "GND" H 5755 3677 50  0000 C CNN
 F 2 "" H 5750 3850 50  0001 C CNN
@@
 GPIO16&17 not exist in ESP32-WROVER.
 Text Label 4150 2350 2    50   ~ 0
+ESP32_IO17
+Text Label 4150 2450 2    50   ~ 0
 ESP32_IO16
-Text Label 4150 2450 2    50   ~ 0
-ESP32_IO17
 Text Label 4350 2450 0    50   ~ 0
 ESP32_IO7
@@
 ESP32_VDD
 $Comp
-L power:GND #PWR07
+L power:GND #PWR08
 U 1 1 5DF02259
 P 1950 4200
-F 0 "#PWR07" H 1950 3950 50  0001 C CNN
+F 0 "#PWR08" H 1950 3950 50  0001 C CNN
 F 1 "GND" H 1955 4027 50  0000 C CNN
 F 2 "" H 1950 4200 50  0001 C CNN
@@
 $EndComp
 $Comp
-L power:GND #PWR08
+L power:GND #PWR09
 U 1 1 5DF04B74
 P 2050 5000
-F 0 "#PWR08" H 2050 4750 50  0001 C CNN
+F 0 "#PWR09" H 2050 4750 50  0001 C CNN
 F 1 "GND" H 2055 4827 50  0000 C CNN
 F 2 "" H 2050 5000 50  0001 C CNN
@@
 $EndComp
 Wire Wire Line
-	1600 5550 800  5550
-Wire Wire Line
 	1600 5650 800  5650
 Wire Wire Line
@@
 Wire Wire Line
 	1600 7250 800  7250
-Text Label 800  5550 0    50   ~ 0
-ESP32_VDD
 Text Label 800  5650 0    50   ~ 0
 ESP32_EN
@@
 Wire Wire Line
 	2700 6550 3500 6550
+Text Label 3500 6550 2    50   ~ 0
+ESP32_IO16
 Text Label 3500 6450 2    50   ~ 0
-ESP32_IO16
-Text Label 3500 6550 2    50   ~ 0
 ESP32_IO17
 $Comp
@@
 $EndComp
 $Comp
-L power:GND #PWR06
+L power:GND #PWR07
 U 1 1 5DE3B3D6
 P 1600 6850
-F 0 "#PWR06" H 1600 6600 50  0001 C CNN
+F 0 "#PWR07" H 1600 6600 50  0001 C CNN
 F 1 "GND" V 1605 6722 50  0000 R CNN
 F 2 "" H 1600 6850 50  0001 C CNN
@@
 $EndComp
 $Comp
-L power:GND #PWR09
+L power:GND #PWR010
 U 1 1 5DE3B79E
 P 2700 5450
-F 0 "#PWR09" H 2700 5200 50  0001 C CNN
+F 0 "#PWR010" H 2700 5200 50  0001 C CNN
 F 1 "GND" V 2705 5322 50  0000 R CNN
 F 2 "" H 2700 5450 50  0001 C CNN
@@
 $EndComp
 $Comp
-L power:GND #PWR010
+L power:GND #PWR011
 U 1 1 5DE3BCC7
 P 2700 6050
-F 0 "#PWR010" H 2700 5800 50  0001 C CNN
+F 0 "#PWR011" H 2700 5800 50  0001 C CNN
 F 1 "GND" V 2705 5922 50  0000 R CNN
 F 2 "" H 2700 6050 50  0001 C CNN
@@
 Text HLabel 8200 1950 0    50   Input ~ 0
 I2S_MCLK
-Text Label 3650 6450 0    50   ~ 0
+Text Label 5900 6800 2    50   ~ 0
 ESP32_IO12
 Wire Wire Line
-	3650 6450 4350 6450
-Text Label 3650 6950 0    50   ~ 0
+	5900 6800 5200 6800
+Text Label 5900 6700 2    50   ~ 0
 ESP32_IO14
 Wire Wire Line
-	3650 6950 4350 6950
-Wire Wire Line
-	4350 6850 4850 6850
-Text Label 3650 6700 0    50   ~ 0
+	5900 6700 5200 6700
+Text Label 5900 7000 2    50   ~ 0
 ESP32_IO15
 Wire Wire Line
-	3650 6700 4350 6700
+	5900 7000 5200 7000
 $Comp
 L Interface_Expansion:TCA9535PWR U3
@@
 ESP32_GPIO33
 $Comp
-L power:GND #PWR016
+L power:GND #PWR015
 U 1 1 5DE8ACE5
 P 9600 6250
-F 0 "#PWR016" H 9600 6000 50  0001 C CNN
+F 0 "#PWR015" H 9600 6000 50  0001 C CNN
 F 1 "GND" H 9605 6077 50  0000 C CNN
 F 2 "" H 9600 6250 50  0001 C CNN
@@
 	9600 4050 9850 4050
 $Comp
-L power:VDD #PWR017
+L power:VDD #PWR016
 U 1 1 5DE92886
 P 10050 4050
-F 0 "#PWR017" H 10050 3900 50  0001 C CNN
+F 0 "#PWR016" H 10050 3900 50  0001 C CNN
 F 1 "VDD" H 10067 4223 50  0000 C CNN
 F 2 "" H 10050 4050 50  0001 C CNN
@@
 Connection ~ 9850 4050
 $Comp
-L power:GND #PWR015
+L power:GND #PWR014
 U 1 1 5DEBE05F
 P 9600 3750
-F 0 "#PWR015" H 9600 3500 50  0001 C CNN
+F 0 "#PWR014" H 9600 3500 50  0001 C CNN
 F 1 "GND" V 9605 3622 50  0000 R CNN
 F 2 "" H 9600 3750 50  0001 C CNN
@@
 Text HLabel 8200 2150 0    50   BiDi ~ 0
 I2S_LR
-$Comp
-L Connector:Conn_01x02_Male J3
-U 1 1 5DED655F
-P 4150 6350
-F 0 "J3" H 4258 6531 50  0000 C CNN
-F 1 "Conn_01x02_Male" H 4258 6440 50  0000 C CNN
-F 2 "Connector_PinHeader_2.54mm:PinHeader_1x02_P2.54mm_Vertical" H 4150 6350 50  0001 C CNN
-F 3 "~" H 4150 6350 50  0001 C CNN
-	1    4150 6350
-	1    0    0    -1
-$EndComp
-$Comp
-L Connector:Conn_01x02_Male J5
-U 1 1 5DED6C65
-P 4150 6850
-F 0 "J5" H 4258 7031 50  0000 C CNN
-F 1 "Conn_01x02_Male" H 4258 6940 50  0000 C CNN
-F 2 "Connector_PinHeader_2.54mm:PinHeader_1x02_P2.54mm_Vertical" H 4150 6850 50  0001 C CNN
-F 3 "~" H 4150 6850 50  0001 C CNN
-	1    4150 6850
-	1    0    0    -1
-$EndComp
-$Comp
-L Connector:Conn_01x02_Male J4
-U 1 1 5DED6EA7
-P 4150 6600
-F 0 "J4" H 4258 6781 50  0000 C CNN
-F 1 "Conn_01x02_Male" H 4258 6690 50  0000 C CNN
-F 2 "Connector_PinHeader_2.54mm:PinHeader_1x02_P2.54mm_Vertical" H 4150 6600 50  0001 C CNN
-F 3 "~" H 4150 6600 50  0001 C CNN
-	1    4150 6600
-	1    0    0    -1
-$EndComp
-$Comp
-L Connector:Conn_ARM_JTAG_SWD_20 J7
-U 1 1 5DEE4A08
-P 6150 6700
-F 0 "J7" H 7000 7350 50  0000 R CNN
-F 1 "Conn_ARM_JTAG_SWD_20" H 7200 7450 50  0000 R CNN
-F 2 "Connector_PinSocket_2.54mm:PinSocket_2x10_P2.54mm_Vertical" H 6600 5650 50  0001 L TNN
-F 3 "http://infocenter.arm.com/help/topic/com.arm.doc.dui0499b/DUI0499B_system_design_reference.pdf" V 5800 5450 50  0001 C CNN
-	1    6150 6700
-	-1   0    0    1
-$EndComp
-Wire Wire Line
-	4350 6350 4850 6350
-NoConn ~ 6150 7500
-$Comp
-L power:GND #PWR013
-U 1 1 5DEF228C
-P 6250 5900
-F 0 "#PWR013" H 6250 5650 50  0001 C CNN
-F 1 "GND" H 6255 5727 50  0000 C CNN
-F 2 "" H 6250 5900 50  0001 C CNN
-F 3 "" H 6250 5900 50  0001 C CNN
-	1    6250 5900
-	-1   0    0    1
-$EndComp
-Wire Wire Line
-	4850 6350 4850 6500
-Wire Wire Line
-	4850 6500 5550 6500
-$Comp
-L Connector:Conn_01x02_Male J6
-U 1 1 5DED67C1
-P 4150 7100
-F 0 "J6" H 4258 7281 50  0000 C CNN
-F 1 "Conn_01x02_Male" H 4258 7190 50  0000 C CNN
-F 2 "Connector_PinHeader_2.54mm:PinHeader_1x02_P2.54mm_Vertical" H 4150 7100 50  0001 C CNN
-F 3 "~" H 4150 7100 50  0001 C CNN
-	1    4150 7100
-	1    0    0    -1
-$EndComp
-Wire Wire Line
-	3650 7200 4350 7200
-Text Label 3650 7200 0    50   ~ 0
+Wire Wire Line
+	5900 6900 5200 6900
+Text Label 5900 6900 2    50   ~ 0
 ESP32_IO13
-Wire Wire Line
-	4350 6600 5550 6600
-Wire Wire Line
-	4850 6850 4850 6700
-Wire Wire Line
-	4850 6700 5550 6700
-Wire Wire Line
-	4950 7100 4950 6800
-Wire Wire Line
-	4950 6800 5550 6800
-Wire Wire Line
-	4350 7100 4950 7100
-NoConn ~ 5550 6900
-NoConn ~ 5550 7200
-NoConn ~ 5550 7100
-NoConn ~ 5550 6300
-NoConn ~ 5550 6200
-Wire Wire Line
-	6250 7500 6250 7550
-$Comp
-L power:VDD #PWR014
-U 1 1 5DF90938
-P 6800 7550
-F 0 "#PWR014" H 6800 7400 50  0001 C CNN
-F 1 "VDD" H 6817 7723 50  0000 C CNN
-F 2 "" H 6800 7550 50  0001 C CNN
-F 3 "" H 6800 7550 50  0001 C CNN
-	1    6800 7550
-	1    0    0    -1
-$EndComp
-Wire Wire Line
-	6250 7550 6800 7550
 Wire Wire Line
 	8200 1950 8750 1950
@@
 Text HLabel 11600 4650 2    50   BiDi ~ 0
 I2S_SCLK
+$Comp
+L power:VDD #PWR06
+U 1 1 5DD6A3F1
+P 1600 5550
+F 0 "#PWR06" H 1600 5400 50  0001 C CNN
+F 1 "VDD" V 1618 5677 50  0000 L CNN
+F 2 "" H 1600 5550 50  0001 C CNN
+F 3 "" H 1600 5550 50  0001 C CNN
+	1    1600 5550
+	0    -1   -1   0
+$EndComp
+Text Notes 5200 6250 0    50   ~ 0
+JTAG only for test in ver 0.
+Text HLabel 8200 2400 0    50   BiDi ~ 0
+EMAC_RMII_TX0
+Text HLabel 8200 2500 0    50   BiDi ~ 0
+EMAC_RMII_TX1
+Text HLabel 8200 2600 0    50   BiDi ~ 0
+EMAC_RMII_TXEN
+Wire Wire Line
+	8200 2400 8750 2400
+Wire Wire Line
+	8200 2500 8750 2500
+Wire Wire Line
+	8200 2600 8750 2600
+Text Label 8750 2500 2    50   ~ 0
+ESP32_GPIO22
+Text Label 8750 2600 2    50   ~ 0
+ESP32_GPIO21
+Text Label 8750 2400 2    50   ~ 0
+ESP32_GPIO19
+Text HLabel 8200 2750 0    50   BiDi ~ 0
+EMAC_RMII_RX0
+Text HLabel 8200 2850 0    50   BiDi ~ 0
+EMAC_RMII_RX1
+Text HLabel 8200 2950 0    50   BiDi ~ 0
+EMAC_RMII_RXDV
+Wire Wire Line
+	8200 2750 8750 2750
+Wire Wire Line
+	8200 2850 8750 2850
+Wire Wire Line
+	8200 2950 8750 2950
+Text Label 8750 2850 2    50   ~ 0
+ESP32_GPIO26
+Text Label 8750 2950 2    50   ~ 0
+ESP32_GPIO27
+Text Label 8750 2750 2    50   ~ 0
+ESP32_GPIO25
+Text HLabel 8200 3100 0    50   BiDi ~ 0
+EMAC_MDIO
+Text HLabel 8200 3200 0    50   BiDi ~ 0
+EMAC_MDC
+Text HLabel 8200 3300 0    50   BiDi ~ 0
+EMAC_REF_CLK
+Wire Wire Line
+	8200 3100 8750 3100
+Wire Wire Line
+	8200 3200 8750 3200
+Wire Wire Line
+	8200 3300 8750 3300
+Text Label 8750 3200 2    50   ~ 0
+ESP32_GPIO13
+Text Label 8750 3300 2    50   ~ 0
+ESP32_GPIO0
+Text Label 8750 3100 2    50   ~ 0
+ESP32_GPIO12
+$Comp
+L Connector:Conn_01x06_Male J3
+U 1 1 5DDA11FE
+P 5000 6800
+F 0 "J3" H 5108 7181 50  0000 C CNN
+F 1 "Conn_01x06_Male" H 5108 7090 50  0000 C CNN
+F 2 "Connector_PinHeader_2.54mm:PinHeader_1x06_P2.54mm_Vertical" H 5000 6800 50  0001 C CNN
+F 3 "~" H 5000 6800 50  0001 C CNN
+	1    5000 6800
+	1    0    0    -1
+$EndComp
+$Comp
+L power:GND #PWR0101
+U 1 1 5DDD8F68
+P 5200 7100
+F 0 "#PWR0101" H 5200 6850 50  0001 C CNN
+F 1 "GND" H 5205 6927 50  0000 C CNN
+F 2 "" H 5200 7100 50  0001 C CNN
+F 3 "" H 5200 7100 50  0001 C CNN
+	1    5200 7100
+	1    0    0    -1
+$EndComp
+$Comp
+L power:VDD #PWR0102
+U 1 1 5DDD95AA
+P 5200 6600
+F 0 "#PWR0102" H 5200 6450 50  0001 C CNN
+F 1 "VDD" H 5217 6773 50  0000 C CNN
+F 2 "" H 5200 6600 50  0001 C CNN
+F 3 "" H 5200 6600 50  0001 C CNN
+	1    5200 6600
+	1    0    0    -1
+$EndComp
+Text Notes 5950 6700 0    50   ~ 0
+MTMS
+Text Notes 5950 6800 0    50   ~ 0
+MTDI
+Text Notes 5950 7000 0    50   ~ 0
+MTDO
+Text Notes 5950 6900 0    50   ~ 0
+MTCK
 $EndSCHEMATC
