File: pwr.sch (KiCad schematic (older format))
At the start: 0 parts

Commit message: 20191113未完工
Parts:
- added C? (x2): 0603_20pF__200_5%_50V, lc_lib:0603_C, symbol lc_Cap:0603_20pF__200_5%_50V
- added C? (x3): 0603_100nF__104_10%_50V, lc_lib:0603_C, symbol lc_Cap:0603_100nF__104_10%_50V
- added C?: 0603_22uF__226_20%_6.3V, lc_lib:0603_C, symbol lc_Cap:0603_22uF__226_20%_6.3V
- added C? (x3): 0805_22uF__226_20%_25V, lc_lib:0805_C, symbol lc_Cap:0805_22uF__226_20%_25V
- added C?: 0603_10uF__106_10%_10V, lc_lib:0603_C, symbol lc_Cap:0603_10uF__106_10%_10V
- added C? (x2): 0603_1uF__105_10%_50V, lc_lib:0603_C, symbol lc_Cap:0603_1uF__105_10%_50V
- added D?: 0603_绿灯, lc_lib:0603_LED_S1, symbol lc_LED:0603_绿灯
- added J?: USB_C_Receptacle_USB2.0, symbol Connector:USB_C_Receptacle_USB2.0
- added L?: L, symbol Device:L
- added R? (x2): 0603_5.1KΩ__5101_1%, lc_lib:0603_R, symbol lc_RES:0603_5.1KΩ__5101_1%
- added R?: 0603_33KΩ__3302_1%, lc_lib:0603_R, symbol lc_RES:0603_33KΩ__3302_1%
- added R?: 0603_10KΩ__1002_1%, lc_lib:0603_R, symbol lc_RES:0603_10KΩ__1002_1%
- added R?: 0603_1.5KΩ__1501_1%, lc_lib:0603_R, symbol lc_RES:0603_1.5KΩ__1501_1%
- added R? (x2): 0603_0Ω__0R0_1%, lc_lib:0603_R, symbol lc_RES:0603_0Ω__0R0_1%
- added R?: 0603_1KΩ__1001_1%, lc_lib:0603_R, symbol lc_RES:0603_1KΩ__1001_1%
- added SW?: SW_Push_DPDT, symbol Switch:SW_Push_DPDT
- added U?: SRV05-4-P-T7_[C85364], lc_lib:SOT-23-6, symbol lc_IC:SRV05-4-P-T7_[C85364]
- added U?: CH340G, Package_SO:SOIC-16_3.9x9.9mm_P1.27mm, symbol Interface_USB:CH340G
- added U?: AOZ1031, Package_SO:SOIC-8_3.9x4.9mm_P1.27mm, symbol AOZ1031:AOZ1031
- added Y?: SMD-3225_4P__12MHZ_20PF_10PPM, lc_lib:SMD-3225_4P, symbol lc_CrystalOscillator:SMD-3225_4P__12MHZ_20PF_10PPM
Connections:
- new net: J?.A4 (VBUS), J?.A9 (VBUS), J?.B4 (VBUS), J?.B9 (VBUS), SW?.5 (B)
- new net: J?.A5 (CC1), R?.1
- new net: J?.B5 (CC2), R?.1
- new net: C?.1, U?.7 (XI), Y?.1 (OSC1)
- new net: C?.1, U?.8 (XO), Y?.3 (OSC2)
- new net: R?.1, U?.5 (COMP)
- new net: L?.1, U?.7 (LX), U?.8 (LX)
- new net: C?.1, C?.1, C?.1, L?.2, R?.1, R?.1
- new net: C?.1, R?.2
- new net: D?.K, R?.1
- new net FB: R?.1, R?.2, U?.4 (FB)
- new net GND: C?.2, C?.2, C?.2, C?.2, C?.2, C?.2, C?.2, C?.2, C?.2, C?.2, C?.2, C?.2, J?.A1 (GND), J?.A12 (GND), J?.B1 (GND), J?.B12 (GND), J?.S1 (SHIELD), R?.2, R?.2, R?.2, R?.2, U?.1 (PGND), U?.2 (GND), U?.3 (AGND), U?.4 (I/O), U?.6 (I/O)
- new net RXD: U?.3 (RXD)
- new net TXD: U?.2 (TXD)
- new net USB+: J?.A6 (D+), J?.B6 (D+), U?.3 (I/O), U?.5 (UD+)
- new net USB-: J?.A7 (D-), J?.B7 (D-), U?.1 (I/O_), U?.6 (UD-)
- new net VBUS: C?.1, C?.1, C?.1, C?.1, SW?.6 (C), U?.2 (VIN), U?.6 (EN)
- new net VDD: C?.1, C?.1, D?.A, R?.1, R?.2, U?.16 (VCC), U?.4 (V3), U?.5 (REF)
- new net VDDA: R?.2
- no-connect marks 0 -> 9

Commit message: 20191113
Parts:
- J9: renamed from J?; footprint (none) -> Connector_USB:USB_C_Receptacle_Palconn_UTC16-G
- gave numbers to parts that had none: 27

Commit message: 20191114
Parts:
- removed SW1: SW_Push_DPDT, symbol Switch:SW_Push_DPDT
- removed U6: SRV05-4-P-T7_[C85364], lc_lib:SOT-23-6, symbol lc_IC:SRV05-4-P-T7_[C85364]
- added U5: SRV05-4, Package_TO_SOT_SMD:SOT-23-6, symbol Power_Protection:SRV05-4
- L1: value L -> 4.7uH; footprint (none) -> Inductor_SMD:L_7.3x7.3_H3.5
- renumbered C19 to C10, C20 to C11, C21 to C12, C22 to C13, C23 to C14, C24 to C15, C25 to C16, C26 to C17, C15 to C6, C16 to C7, C17 to C8, C18 to C9, J9 to J7, R20 to R10, R13 to R3, R14 to R4, R15 to R5, R16 to R6, R17 to R7, R18 to R8, R19 to R9, U5 to U4, U7 to U6, Y2 to Y1
Connections:
- net GND: now also U5.2 (VN)
- net USB+: now also U5.6 (IO4)
- net USB-: now also U5.1 (IO1)
- net VBUS: now also J7.A4 (VBUS), J7.A9 (VBUS), J7.B4 (VBUS), J7.B9 (VBUS)
- net VDD: now also U5.5 (VP)
