File: sensors.sch (KiCad schematic (older format))
At the start: 2 parts, among them U8 MPU-6050, U9 BMP280

Commit message: 20191114
Parts:
- added C24, C25, C26, C28, C29: 0603_100nF__104_10%_50V, lc_lib:0603_C, symbol lc_Cap:0603_100nF__104_10%_50V
- added C27: 0603_2.2nF__222_10%_50V, lc_lib:0603_C, symbol lc_Cap:0603_2.2nF__222_10%_50V
- renumbered U8 to U7, U9 to U8
Connections:
- net at U7.10 (REGOUT): now also C26.1
- net MPU6050_INT: now reaches U7.12 (INT)
- net VDDA: now reaches U7.13 (VDD)
- net VDDA: now also U8.8 (VDD), C25.1, C29.1
- net GND: now reaches U7.18 (GND)
- net GND: now also U7.9 (AD0), U8.1 (GND), U8.5 (SDO), U8.7 (GND), C24.2, C25.2, C26.2, C27.2, C28.2, C29.2
- net at U7.20 (CPOUT): now also C27.1
- net MPU6050_I2C_SCL: now reaches U7.23 (SCL)
- net MPU6050_I2C_SDA: now reaches U7.24 (SDA)
- net VDD: now reaches U7.8 (VDDIO)
- net VDD: now also U8.2 (CSB), U8.6 (VDDIO), C24.1, C28.1
- net BMP280_I2C_SDA: now reaches U8.3 (SDI)
- net BMP280_I2C_SCL: now reaches U8.4 (SCK)
- no-connect marks 0 -> 4
Other:
- note added: "I2C ADDR: 0b1110110X"
- note added: "I2C ADDR:0b1101000X"
- moved on the sheet: U8
